Commit message: Adaptation to EtherCAT comm & RCL

File: kortex_description/arms/linkm/7dof/urdf/kortex.ros2_control.xacro (robot description, xacro)
@@ -24,5 +24,18 @@
     gripper_max_velocity:=100.0
     gripper_max_force:=100.0
-    moveit_active:=false">
+    moveit_active:=false
+    ethercat_lib_path:=/usr/local/lib/libethercat.so
+    network_topology_file:=USE_PACKAGE_DEFAULT
+    arm_part_number:=ARM-L3M000-001
+    arm_part_number_revision:=A
+    arm_serial_number:=0001
+    arm_nb_actuators:=7
+    slave_pos_range_min:=0
+    slave_pos_range_max:=13
+    network_thread_cpu_core:=-1
+    control_thread_cpu_core:=-1
+    gravity_x:=0.0
+    gravity_y:=0.0
+    gravity_z:=-9.81">
     <ros2_control name="${name}" type="system">
       <hardware>
@@ -44,18 +57,27 @@
         </xacro:if>
         <xacro:unless value="${use_fake_hardware or sim_gazebo or sim_ignition or sim_isaac}">
+          <!-- KIMA over EtherCAT via Kinova's Robot Control Library (RCL). -->
           <plugin>kortex_driver/KortexMultiInterfaceHardware</plugin>
-          <param name="robot_ip">${robot_ip}</param>
-          <param name="username">${username}</param>
-          <param name="password">${password}</param>
-          <param name="port">${port}</param>
-          <param name="port_realtime">${port_realtime}</param>
-          <param name="session_inactivity_timeout_ms">${session_inactivity_timeout_ms}</param>
-          <param name="connection_inactivity_timeout_ms">${connection_inactivity_timeout_ms}</param>
-          <param name="tf_prefix">"${tf_prefix}"</param>
+          <param name="ethercat_lib_path">${ethercat_lib_path}</param>
+          <!-- Default to the topology shipped with kortex_description; override
+               by passing network_topology_file to the macro. -->
+          <xacro:if value="${network_topology_file == 'USE_PACKAGE_DEFAULT'}">
+            <param name="network_topology_file">$(find kortex_description)/arms/linkm/7dof/config/network_topology_1_arm.yaml</param>
+          </xacro:if>
+          <xacro:unless value="${network_topology_file == 'USE_PACKAGE_DEFAULT'}">
+            <param name="network_topology_file">${network_topology_file}</param>
+          </xacro:unless>
+          <param name="arm_part_number">${arm_part_number}</param>
+          <param name="arm_part_number_revision">${arm_part_number_revision}</param>
+          <param name="arm_serial_number">${arm_serial_number}</param>
+          <param name="arm_nb_actuators">${arm_nb_actuators}</param>
+          <param name="slave_pos_range_min">${slave_pos_range_min}</param>
+          <param name="slave_pos_range_max">${slave_pos_range_max}</param>
+          <param name="network_thread_cpu_core">${network_thread_cpu_core}</param>
+          <param name="control_thread_cpu_core">${control_thread_cpu_core}</param>
+          <param name="gravity_x">${gravity_x}</param>
+          <param name="gravity_y">${gravity_y}</param>
+          <param name="gravity_z">${gravity_z}</param>
           <param name="prefix">${prefix}</param>
-          <param name="use_internal_bus_gripper_comm">${use_internal_bus_gripper_comm}</param>
-          <param name="gripper_joint_name">${gripper_joint_name}</param>
-          <param name="gripper_max_velocity">${gripper_max_velocity}</param>
-          <param name="gripper_max_force">${gripper_max_force}</param>
         </xacro:unless>
       </hardware>
@@ -144,13 +166,7 @@
         <state_interface name="effort"/>
       </joint>
-      <xacro:unless value="${use_fake_hardware or sim_gazebo or sim_ignition or sim_isaac}">
-        <xacro:if value="${use_internal_bus_gripper_comm}">
-          <joint name="${prefix}${gripper_joint_name}">
-            <command_interface name="position" />
-            <state_interface name="position"/>
-            <state_interface name="velocity"/>
-          </joint>
-        </xacro:if>
-      </xacro:unless>
+      <!-- No gripper: KIMA is arm-only on the EtherCAT bus and the RCL API has
+           no gripper command path. The gripper (mock) joint is only kept for
+           the simulation/fake-hardware plugins above. -->
     </ros2_control>
   </xacro:macro>
