Commit message: comprehensive clean up 2

File: kortex_description/arms/kima/7dof/urdf/kima_macro.xacro (robot description, xacro)
@@ -1,5 +1,5 @@
 <?xml version="1.0"?>
-<robot name="linkm_arm" xmlns:xacro="http://ros.org/wiki/xacro">
-  <!-- last_arm_link is read by kortex_robot.xacro to attach the gripper or tool_frame -->
+<robot name="kima_arm" xmlns:xacro="http://ros.org/wiki/xacro">
+  <!-- last_arm_link is read by kortex_robot.xacro to attach the tool_frame -->
   <xacro:property name="last_arm_link" value="end_effector_link"/>
   <xacro:property name="PI" value="3.1415926535897931"/>
@@ -17,8 +17,4 @@
     session_inactivity_timeout_ms:=6000
     connection_inactivity_timeout_ms:=2000
-    use_internal_bus_gripper_comm:=true
-    gripper_joint_name
-    gripper_max_velocity:=100.0
-    gripper_max_force:=100.0
     use_fake_hardware:=false
     fake_sensor_commands:=false
@@ -32,5 +28,5 @@
     moveit_active:=false">
     <!-- ros2 control include -->
-    <xacro:include filename="$(find kortex_description)/arms/linkm/7dof/urdf/kortex.ros2_control.xacro" />
+    <xacro:include filename="$(find kortex_description)/arms/kima/7dof/urdf/kortex.ros2_control.xacro" />
     <xacro:kortex_ros2_control
       name="${prefix}KortexMultiInterfaceHardware"
@@ -51,9 +47,5 @@
       port_realtime="${port_realtime}"
       session_inactivity_timeout_ms="${session_inactivity_timeout_ms}"
-      connection_inactivity_timeout_ms="${connection_inactivity_timeout_ms}"
-      use_internal_bus_gripper_comm="${use_internal_bus_gripper_comm}"
-      gripper_max_velocity="${gripper_max_velocity}"
-      gripper_max_force="${gripper_max_force}"
-      gripper_joint_name="${gripper_joint_name}"/>
+      connection_inactivity_timeout_ms="${connection_inactivity_timeout_ms}"/>
     <!-- Fixed joint attaching arm base to parent link -->
     <joint name="${prefix}base_joint" type="fixed">
@@ -72,5 +64,5 @@
         <origin xyz="0 0 0" rpy="0 0 0" />
         <geometry>
-          <mesh filename="file://$(find kortex_description)/arms/linkm/urdf/meshes/base_link.STL" />
+          <mesh filename="file://$(find kortex_description)/arms/kima/urdf/meshes/base_link.STL" />
         </geometry>
         <material name="">
@@ -101,5 +93,5 @@
         <origin xyz="0 0 0" rpy="0 0 0" />
         <geometry>
-          <mesh filename="file://$(find kortex_description)/arms/linkm/urdf/meshes/j1-j2_link.STL" />
+          <mesh filename="file://$(find kortex_description)/arms/kima/urdf/meshes/j1-j2_link.STL" />
         </geometry>
         <material name="">
@@ -137,5 +129,5 @@
         <origin xyz="0 0 0" rpy="0 0 0" />
         <geometry>
-          <mesh filename="file://$(find kortex_description)/arms/linkm/urdf/meshes/j2-j3_link.STL" />
+          <mesh filename="file://$(find kortex_description)/arms/kima/urdf/meshes/j2-j3_link.STL" />
         </geometry>
         <material name="">
@@ -181,5 +173,5 @@
         <origin xyz="0 0 0" rpy="0 0 0" />
         <geometry>
-          <mesh filename="file://$(find kortex_description)/arms/linkm/urdf/meshes/j3-j4_link.STL" />
+          <mesh filename="file://$(find kortex_description)/arms/kima/urdf/meshes/j3-j4_link.STL" />
         </geometry>
         <material name="">
@@ -225,5 +217,5 @@
         <origin xyz="0 0 0" rpy="0 0 0" />
         <geometry>
-          <mesh filename="file://$(find kortex_description)/arms/linkm/urdf/meshes/j4-j5_link.STL" />
+          <mesh filename="file://$(find kortex_description)/arms/kima/urdf/meshes/j4-j5_link.STL" />
         </geometry>
         <material name="">
@@ -273,5 +265,5 @@
         <origin xyz="0 0 0" rpy="0 0 0" />
         <geometry>
-          <mesh filename="file://$(find kortex_description)/arms/linkm/urdf/meshes/j5-j6_link.STL" />
+          <mesh filename="file://$(find kortex_description)/arms/kima/urdf/meshes/j5-j6_link.STL" />
         </geometry>
         <material name="">
@@ -309,5 +301,5 @@
         <origin xyz="0 0 0" rpy="0 0 0" />
         <geometry>
-          <mesh filename="file://$(find kortex_description)/arms/linkm/urdf/meshes/j6-j7_link.STL" />
+          <mesh filename="file://$(find kortex_description)/arms/kima/urdf/meshes/j6-j7_link.STL" />
         </geometry>
         <material name="">
@@ -345,5 +337,5 @@
         <origin xyz="0 0 0" rpy="0 0 0" />
         <geometry>
-          <mesh filename="file://$(find kortex_description)/arms/linkm/urdf/meshes/j7-tif_link.STL" />
+          <mesh filename="file://$(find kortex_description)/arms/kima/urdf/meshes/j7-tif_link.STL" />
         </geometry>
         <material name="">

File: kortex_description/arms/kima/7dof/urdf/kortex.ros2_control.xacro (robot description, xacro)
@@ -11,5 +11,4 @@
     isaac_joint_commands:=/isaac_joint_commands
     isaac_joint_states:=/isaac_joint_states
-    use_internal_bus_gripper_comm:=true
     tf_prefix
     initial_positions:=${dict(joint_1=0.0,joint_2=0.0,joint_3=0.0,joint_4=0.0,joint_5=0.0,joint_6=0.0,joint_7=0.0)}
@@ -21,7 +20,4 @@
     session_inactivity_timeout_ms
     connection_inactivity_timeout_ms
-    gripper_joint_name
-    gripper_max_velocity:=100.0
-    gripper_max_force:=100.0
     moveit_active:=false
     ethercat_lib_path:=/usr/local/lib/libethercat.so
@@ -44,5 +40,5 @@
         </xacro:if>
         <xacro:if value="${sim_ignition}">
-          <plugin>ign_ros2_control/IgnitionSystem</plugin>
+          <plugin>gz_ros2_control/GazeboSimSystem</plugin>
         </xacro:if>
         <xacro:if value="${sim_isaac}">
@@ -63,5 +59,5 @@
                by passing network_topology_file to the macro. -->
           <xacro:if value="${network_topology_file == 'USE_PACKAGE_DEFAULT'}">
-            <param name="network_topology_file">$(find kortex_description)/arms/linkm/7dof/config/network_topology_1_arm.yaml</param>
+            <param name="network_topology_file">$(find kortex_description)/arms/kima/7dof/config/network_topology_1_arm.yaml</param>
           </xacro:if>
           <xacro:unless value="${network_topology_file == 'USE_PACKAGE_DEFAULT'}">
@@ -172,7 +168,4 @@
         <state_interface name="effort"/>
       </joint>
-      <!-- No gripper: KIMA is arm-only on the EtherCAT bus and the RCL API has
-           no gripper command path. The gripper (mock) joint is only kept for
-           the simulation/fake-hardware plugins above. -->
     </ros2_control>
   </xacro:macro>

File: kortex_description/multiple_robots/kortex_dual_robots.xacro (robot description, xacro)
@@ -2,5 +2,4 @@
 <robot name="dual_robot" xmlns:xacro="http://ros.org/wiki/xacro">
     <xacro:arg name="left_arm"  default=""/>
-    <xacro:arg name="left_gripper" default=""/>
     <xacro:arg name="left_dof"  default=""/>
     <xacro:arg name="left_vision" default=""/>
@@ -8,5 +7,4 @@
     <xacro:arg name="left_prefix" default=""/>
     <xacro:arg name="right_arm"  default=""/>
-    <xacro:arg name="right_gripper" default=""/>
     <xacro:arg name="right_dof"  default=""/>
     <xacro:arg name="right_vision" default=""/>
@@ -29,5 +27,4 @@
     <xacro:load_robot
         arm="$(arg left_arm)"
-        gripper="$(arg left_gripper)"
         dof="$(arg left_dof)"
         vision="$(arg left_vision)"
@@ -37,5 +34,4 @@
     <xacro:load_robot
         arm="$(arg right_arm)"
-        gripper="$(arg right_gripper)"
         dof="$(arg right_dof)"
         vision="$(arg right_vision)"

File: kortex_description/robots/kima.xacro (robot description, xacro)
@@ -1,6 +1,6 @@
 <?xml version="1.0"?>
-<robot name="linkm" xmlns:xacro="http://ros.org/wiki/xacro">
+<robot name="kima" xmlns:xacro="http://ros.org/wiki/xacro">
     <!-- Arguments -->
-    <xacro:arg name="arm" default="linkm" />
+    <xacro:arg name="arm" default="kima" />
     <xacro:arg name="dof" default="7" />
     <xacro:arg name="vision" default="false" />
@@ -12,8 +12,4 @@
     <xacro:arg name="session_inactivity_timeout_ms" default="60000" />
     <xacro:arg name="connection_inactivity_timeout_ms" default="2000" />
-    <xacro:arg name="gripper" default="" />
-    <xacro:arg name="gripper_joint_name" default="finger_joint" />
-    <xacro:arg name="gripper_max_velocity" default="100.0" />
-    <xacro:arg name="gripper_max_force" default="100.0" />
     <xacro:arg name="sim_gazebo" default="false" />
     <xacro:arg name="sim_ignition" default="false" />
@@ -22,5 +18,4 @@
     <xacro:arg name="use_fake_hardware" default="false" />
     <xacro:arg name="fake_sensor_commands" default="false" />
-    <xacro:arg name="use_internal_bus_gripper_comm" default="false" />
     <xacro:arg name="use_external_cable" default="false" />
     <xacro:include filename="$(find kortex_description)/robots/kortex_robot.xacro" />
@@ -33,8 +28,4 @@
         parent="world"
         arm="$(arg arm)"
-        gripper="$(arg gripper)"
-        gripper_joint_name="$(arg gripper_joint_name)"
-        gripper_max_velocity="$(arg gripper_max_velocity)"
-        gripper_max_force="$(arg gripper_max_force)"
         dof="$(arg dof)"
         vision="$(arg vision)"
@@ -46,5 +37,4 @@
         session_inactivity_timeout_ms="$(arg session_inactivity_timeout_ms)"
         connection_inactivity_timeout_ms="$(arg connection_inactivity_timeout_ms)"
-        use_internal_bus_gripper_comm="$(arg use_internal_bus_gripper_comm)"
         prefix="$(arg prefix)"
         use_fake_hardware="$(arg use_fake_hardware)"

File: kortex_description/robots/kinova.urdf.xacro (robot description, xacro)
@@ -15,9 +15,4 @@
   <xacro:arg name="session_inactivity_timeout_ms" default="60000" />
   <xacro:arg name="connection_inactivity_timeout_ms" default="2000" />
-  <xacro:arg name="gripper" default="" />
-  <xacro:arg name="gripper_joint_name" default="finger_joint" />
-  <xacro:arg name="gripper_max_velocity" default="100.0" />
-  <xacro:arg name="gripper_max_force" default="100.0" />
-  <xacro:arg name="use_internal_bus_gripper_comm" default="false" />
   <xacro:arg name="use_fake_hardware" default="false" />
   <xacro:arg name="fake_sensor_commands" default="false" />
@@ -29,5 +24,5 @@
   <xacro:arg name="camera_height" default="480"/>
   <xacro:arg name="camera_fps" default="6"/>
-  <xacro:arg name="simulation_controllers" default="$(find kortex_description)/arm/$(arg arm)/$(arg dof)dof/config/ros2_controllers.yaml" />
+  <xacro:arg name="simulation_controllers" default="$(find kortex_description)/arms/$(arg arm)/$(arg dof)dof/config/ros2_controllers.yaml" />
   <xacro:arg name="moveit_active" default="false"/>
   <!-- import main macro -->
@@ -42,8 +37,4 @@
     parent="world"
     arm="$(arg arm)"
-    gripper="$(arg gripper)"
-    gripper_joint_name="$(arg gripper_joint_name)"
-    gripper_max_velocity="$(arg gripper_max_velocity)"
-    gripper_max_force="$(arg gripper_max_force)"
     dof="$(arg dof)"
     vision="$(arg vision)"
@@ -55,5 +46,4 @@
     session_inactivity_timeout_ms="$(arg session_inactivity_timeout_ms)"
     connection_inactivity_timeout_ms="$(arg connection_inactivity_timeout_ms)"
-    use_internal_bus_gripper_comm="$(arg use_internal_bus_gripper_comm)"
     prefix="$(arg prefix)"
     use_fake_hardware="$(arg use_fake_hardware)"
@@ -81,9 +71,9 @@
     </gazebo>
     <gazebo>
-      <plugin filename="libign_ros2_control-system.so" name="ign_ros2_control::IgnitionROS2ControlPlugin">
+      <plugin filename="gz_ros2_control-system" name="gz_ros2_control::GazeboSimROS2ControlPlugin">
         <parameters>$(arg simulation_controllers)</parameters>
         <controller_manager_node_name>$(arg prefix)controller_manager</controller_manager_node_name>
       </plugin>
-      <plugin filename="libignition-gazebo-sensors-system.so" name="ignition::gazebo::systems::Sensors">
+      <plugin filename="gz-sim-sensors-system" name="gz::sim::systems::Sensors">
         <render_engine>$(arg gazebo_renderer)</render_engine>
       </plugin>

File: kortex_description/robots/kortex_robot.xacro (robot description, xacro)
@@ -6,6 +6,4 @@
     prefix
     arm
-    gripper
-    gripper_joint_name
     dof
     vision
@@ -17,5 +15,4 @@
     session_inactivity_timeout_ms
     connection_inactivity_timeout_ms
-    use_internal_bus_gripper_comm:=false
     use_fake_hardware:=false
     fake_sensor_commands:=false
@@ -27,7 +24,4 @@
     use_external_cable:=false
     initial_positions:=${dict(joint_1=0.0,joint_2=0.0,joint_3=0.0,joint_4=0.0,joint_5=0.0,joint_6=0.0,joint_7=0.0)}
-    gripper_max_velocity:=100.0
-    gripper_max_force:=100.0
-    gripper_com_port:=/dev/ttyUSB0
     moveit_active:=false">
     <!-- Include and load arm macro files -->
@@ -46,5 +40,4 @@
       connection_inactivity_timeout_ms="${connection_inactivity_timeout_ms}"
       prefix="${prefix}"
-      use_internal_bus_gripper_comm="${use_internal_bus_gripper_comm}"
       use_fake_hardware="${use_fake_hardware}"
       fake_sensor_commands="${fake_sensor_commands}"
@@ -54,7 +47,4 @@
       isaac_joint_commands="${isaac_joint_commands}"
       isaac_joint_states="${isaac_joint_states}"
-      gripper_joint_name="${gripper_joint_name}"
-      gripper_max_velocity="${gripper_max_velocity}"
-      gripper_max_force="${gripper_max_force}"
       use_external_cable="${use_external_cable}"
       initial_positions="${initial_positions}"
@@ -62,31 +52,12 @@
       <xacro:insert_block name="origin" />
     </xacro:load_arm>
-    <!-- If no gripper, define tool frame here -->
-    <xacro:if value="${not gripper}">
-      <link name="${prefix}tool_frame"/>
-      <joint name="${prefix}tool_frame_joint" type="fixed">
-        <origin xyz="0 0 0" rpy="0 0 0" />
-        <parent link="${prefix}${last_arm_link}" />
-        <child link="${prefix}tool_frame" />
-        <axis xyz="0 0 0" />
-      </joint>
-    </xacro:if>
-    <!-- Include and load the gripper if defined -->
-    <xacro:unless value="${not gripper}">
-      <xacro:include filename="$(find kortex_description)/grippers/${gripper}/urdf/${gripper}_macro.xacro" />
-      <!-- last_arm_link is defined in "$(find kortex_description)/arms/${arm}/urdf/${arm}_macro.xacro" -->
-      <xacro:load_gripper
-        parent="${prefix}${last_arm_link}"
-        prefix="${prefix}"
-        use_fake_hardware="${use_fake_hardware}"
-        fake_sensor_commands="${fake_sensor_commands}"
-        sim_ignition="${sim_ignition}"
-        sim_isaac="${sim_isaac}"
-        isaac_joint_commands="${isaac_joint_commands}"
-        isaac_joint_states="${isaac_joint_states}"
-        com_port="${gripper_com_port}"
-        use_internal_bus_gripper_comm="${use_internal_bus_gripper_comm}"
-        moveit_active="${moveit_active}"/>
-    </xacro:unless>
+    <!-- Tool frame at the end of the arm -->
+    <link name="${prefix}tool_frame"/>
+    <joint name="${prefix}tool_frame_joint" type="fixed">
+      <origin xyz="0 0 0" rpy="0 0 0" />
+      <parent link="${prefix}${last_arm_link}" />
+      <child link="${prefix}tool_frame" />
+      <axis xyz="0 0 0" />
+    </joint>
   </xacro:macro>
 </robot>
